Commit message: URDF: Lidar-Position korrigiert (hinten, höher)

File: ros2_ws/src/amr_description/urdf/amr.urdf (robot description, URDF)
Before this commit: robot amr, 3 links, 2 joints
Links:
- link base_link: geometry collision box size=0.20 0.18 0.04; visual box size=0.20 0.18 0.04
- link laser: geometry collision cylinder length=0.04 radius=0.035; visual cylinder length=0.04 radius=0.035
Joints:
- joint base_link_to_laser: origin xyz=0.08 0 0.08 rpy=0 0 0 -> xyz=-0.07 0 0.13 rpy=0 0 0

Commit message: URDF: Lidar 180° Rotation korrigiert

File: ros2_ws/src/amr_description/urdf/amr.urdf (robot description, URDF)
Before this commit: robot amr, 3 links, 2 joints
Joints:
- joint base_link_to_laser: origin xyz=-0.07 0 0.13 rpy=0 0 0 -> xyz=-0.07 0 0.13 rpy=0 0 3.14159
